File: Power_Breakout/Power_Breakout.sch (KiCad schematic (older format))
At the start: 5 parts, among them J1 12v Out, J2 GND Out, J3 PS Conn, SW1 ON

Commit message: added more text to silkscreen
Parts:
- SW1: symbol Switch:SW_SPST -> Switch:SW_SPDT
Connections:
- net at J3.33 (Pin_33): now also SW1.3 (C); no longer SW1.1 (A)
- no-connect marks 10 -> 11
Other:
- moved on the sheet: R1
Changed lines of the file:
@@
 L Device:R R1
 U 1 1 5E2A6BED
-P 7440 4930
-F 0 "R1" H 7510 4976 50  0000 L CNN
-F 1 "110" H 7510 4885 50  0000 L CNN
-F 2 "Resistor_THT:R_Axial_DIN0207_L6.3mm_D2.5mm_P7.62mm_Horizontal" V 7370 4930 50  0001 C CNN
-F 3 "~" H 7440 4930 50  0001 C CNN
-	1    7440 4930
-	1    0    0    -1
-$EndComp
-Wire Wire Line
-	7440 4780 7040 4780
+P 7595 4930
+F 0 "R1" H 7665 4976 50  0000 L CNN
+F 1 "110" H 7665 4885 50  0000 L CNN
+F 2 "Resistor_THT:R_Axial_DIN0207_L6.3mm_D2.5mm_P7.62mm_Horizontal" V 7525 4930 50  0001 C CNN
+F 3 "~" H 7595 4930 50  0001 C CNN
+	1    7595 4930
+	1    0    0    -1
+$EndComp
+Wire Wire Line
+	7595 4780 7040 4780
 Wire Wire Line
 	6540 2080 6540 2180
@@
 Connection ~ 5245 3445
 $Comp
-L Switch:SW_SPST SW1
+L Switch:SW_SPDT SW1
 U 1 1 5E2C1445
-P 7240 5080
-F 0 "SW1" H 7240 5315 50  0000 C CNN
-F 1 "ON" H 7240 5224 50  0000 C CNN
-F 2 "switch:switch_mmp122-r" H 7240 5080 50  0001 C CNN
-F 3 "~" H 7240 5080 50  0001 C CNN
-	1    7240 5080
-	1    0    0    -1
+P 7240 5180
+F 0 "SW1" H 7240 5415 50  0000 C CNN
+F 1 "ON" H 7240 5324 50  0000 C CNN
+F 2 "switch:switch_mmp122-r" H 7240 5180 50  0001 C CNN
+F 3 "~" H 7240 5180 50  0001 C CNN
+	1    7240 5180
+	-1   0    0    1
 $EndComp
 NoConn ~ 7040 4580
@@
 Wire Wire Line
 	4610 2325 4725 2325
+Wire Wire Line
+	7440 5180 7595 5180
+Wire Wire Line
+	7595 5180 7595 5080
+NoConn ~ 7040 5280
 $EndSCHEMATC
