File: PiHat/PiHat.sch (KiCad schematic (older format))
At the start: 31 parts, among them J1 Raspberry_Pi_2_3, J2 PWR_IN, J3 VIN Voltage, J4 String 1, J5 String 2, J6 RTC Conn, J7 DMX Out, J8 OLED, J9 GPIO, U1 74HC125, U2 OKI-78SR-5, U3 SP3485CP

Commit message: added BOM and Added serial port silkscreen
Parts:
- C1, C2: Digi-Key_PN (none) -> 493-1103-ND; MPN (none) -> UVR1H100MDD
- C3, C4: Digi-Key_PN (none) -> 478-7336-1-ND; MPN (none) -> SR215C104KARTR1
- J1: Digi-Key_PN (none) -> S7123-ND; MPN (none) -> PPPC202LFBN-RC
- J7: Digi-Key_PN (none) -> 277-5738-ND/277-2418-ND; MPN (none) -> 1843622/1840382
- J8, J9: Digi-Key_PN (none) -> S7002-ND; MPN (none) -> PPTC041LFBN-RC
- R1, R2: Digi-Key_PN (none) -> CF14JT33R0CT-ND; MPN (none) -> CF14JT33R0
- R3, R5: Digi-Key_PN (none) -> CF14JT120RCT-ND; MPN (none) -> CF14JT120R
- R4: Digi-Key_PN (none) -> CF14JT10K0CT-ND; MPN (none) -> CF14JT10K0
- U3: Digi-Key_PN (none) -> MAX14780EEPA+-ND; MPN (none) -> MAX14780EEPA+
Changed lines of the file:
@@
 F 2 "Connector_PinSocket_2.54mm:PinSocket_2x20_P2.54mm_Vertical" H 2390 4910 50  0001 C CNN
 F 3 "https://www.raspberrypi.org/documentation/hardware/raspberrypi/schematics/rpi_SCH_3bplus_1p0_reduced.pdf" H 2390 4910 50  0001 C CNN
+F 4 "S7123-ND" H 2390 4910 50  0001 C CNN "Digi-Key_PN"
+F 5 "PPPC202LFBN-RC" H 2390 4910 50  0001 C CNN "MPN"
 	1    2390 4910
 	1    0    0    -1
@@
 F 2 "Resistor_THT:R_Axial_DIN0207_L6.3mm_D2.5mm_P7.62mm_Horizontal" V 5070 4890 50  0001 C CNN
 F 3 "~" H 5140 4890 50  0001 C CNN
+F 4 "CF14JT33R0CT-ND" H 5140 4890 50  0001 C CNN "Digi-Key_PN"
+F 5 "CF14JT33R0" H 5140 4890 50  0001 C CNN "MPN"
 	1    5140 4890
 	0    1    1    0
@@
 F 2 "Resistor_THT:R_Axial_DIN0207_L6.3mm_D2.5mm_P7.62mm_Horizontal" V 5580 5390 50  0001 C CNN
 F 3 "~" H 5650 5390 50  0001 C CNN
+F 4 "CF14JT33R0CT-ND" H 5650 5390 50  0001 C CNN "Digi-Key_PN"
+F 5 "CF14JT33R0" H 5650 5390 50  0001 C CNN "MPN"
 	1    5650 5390
 	0    1    1    0
@@
 F 2 "Resistor_THT:R_Axial_DIN0207_L6.3mm_D2.5mm_P7.62mm_Horizontal" V 9420 5030 50  0001 C CNN
 F 3 "~" H 9490 5030 50  0001 C CNN
+F 4 "CF14JT120RCT-ND" H 9490 5030 50  0001 C CNN "Digi-Key_PN"
+F 5 "CF14JT120R" H 9490 5030 50  0001 C CNN "MPN"
 	1    9490 5030
 	1    0    0    -1
@@
 F 2 "Package_DIP:DIP-8_W7.62mm" H 8890 5030 50  0001 C CIN
 F 3 "http://www.icbase.com/pdf/SPX/SPX00480106.pdf" H 8890 5030 50  0001 C CNN
+F 4 "MAX14780EEPA+-ND" H 8890 5030 50  0001 C CNN "Digi-Key_PN"
+F 5 "MAX14780EEPA+" H 8890 5030 50  0001 C CNN "MPN"
 	1    8890 5030
 	1    0    0    -1
@@
 F 2 "Connector_Phoenix_MC:PhoenixContact_MCV_1,5_4-G-3.5_1x04_P3.50mm_Vertical" H 10090 4930 50  0001 C CNN
 F 3 "~" H 10090 4930 50  0001 C CNN
+F 4 "277-5738-ND/277-2418-ND" H 10090 4930 50  0001 C CNN "Digi-Key_PN"
+F 5 "1843622/1840382" H 10090 4930 50  0001 C CNN "MPN"
 	1    10090 4930
 	1    0    0    -1
@@
 F 2 "Resistor_THT:R_Axial_DIN0207_L6.3mm_D2.5mm_P7.62mm_Horizontal" V 8310 4980 50  0001 C CNN
 F 3 "~" H 8380 4980 50  0001 C CNN
+F 4 "CF14JT10K0CT-ND" H 8380 4980 50  0001 C CNN "Digi-Key_PN"
+F 5 "CF14JT10K0" H 8380 4980 50  0001 C CNN "MPN"
 	1    8380 4980
 	1    0    0    -1
@@
 F 2 "Capacitor_THT:C_Rect_L7.0mm_W2.0mm_P5.00mm" H 6548 4660 50  0001 C CNN
 F 3 "~" H 6510 4810 50  0001 C CNN
+F 4 "478-7336-1-ND" H 6510 4810 50  0001 C CNN "Digi-Key_PN"
+F 5 "SR215C104KARTR1" H 6510 4810 50  0001 C CNN "MPN"
 	1    6510 4810
 	1    0    0    -1
@@
 F 2 "Capacitor_THT:C_Rect_L7.0mm_W2.0mm_P5.00mm" H 9298 4310 50  0001 C CNN
 F 3 "~" H 9260 4460 50  0001 C CNN
+F 4 "478-7336-1-ND" H 9260 4460 50  0001 C CNN "Digi-Key_PN"
+F 5 "SR215C104KARTR1" H 9260 4460 50  0001 C CNN "MPN"
 	1    9260 4460
 	1    0    0    -1
@@
 F 2 "Capacitor_THT:CP_Radial_D5.0mm_P2.00mm" H 3738 1770 50  0001 C CNN
 F 3 "~" H 3700 1920 50  0001 C CNN
+F 4 "493-1103-ND" H 3700 1920 50  0001 C CNN "Digi-Key_PN"
+F 5 "UVR1H100MDD" H 3700 1920 50  0001 C CNN "MPN"
 	1    3700 1920
 	1    0    0    -1
@@
 F 2 "Capacitor_THT:CP_Radial_D5.0mm_P2.00mm" H 4418 1770 50  0001 C CNN
 F 3 "~" H 4380 1920 50  0001 C CNN
+F 4 "493-1103-ND" H 4380 1920 50  0001 C CNN "Digi-Key_PN"
+F 5 "UVR1H100MDD" H 4380 1920 50  0001 C CNN "MPN"
 	1    4380 1920
 	1    0    0    -1
@@
 F 2 "Resistor_THT:R_Axial_DIN0207_L6.3mm_D2.5mm_P7.62mm_Horizontal" V 4990 2120 50  0001 C CNN
 F 3 "~" H 5060 2120 50  0001 C CNN
+F 4 "CF14JT120RCT-ND" H 5060 2120 50  0001 C CNN "Digi-Key_PN"
+F 5 "CF14JT120R" H 5060 2120 50  0001 C CNN "MPN"
 	1    5060 2120
 	1    0    0    -1
@@
 F 2 "Connector_PinSocket_2.54mm:PinSocket_1x04_P2.54mm_Vertical" H 6650 2310 50  0001 C CNN
 F 3 "~" H 6650 2310 50  0001 C CNN
+F 4 "S7002-ND" H 6650 2310 50  0001 C CNN "Digi-Key_PN"
+F 5 "PPTC041LFBN-RC" H 6650 2310 50  0001 C CNN "MPN"
 	1    6650 2310
 	-1   0    0    -1
@@
 F 2 "Connector_PinSocket_2.54mm:PinSocket_1x04_P2.54mm_Vertical" H 6640 3120 50  0001 C CNN
 F 3 "~" H 6640 3120 50  0001 C CNN
+F 4 "S7002-ND" H 6640 3120 50  0001 C CNN "Digi-Key_PN"
+F 5 "PPTC041LFBN-RC" H 6640 3120 50  0001 C CNN "MPN"
 	1    6640 3120
 	-1   0    0    -1
