File: Power_Distribution/Power_Distribution.sch (KiCad schematic (older format))
At the start: 14 parts, among them J1 PWR Out, J2 GND Out

Commit message: Update Silkscreen and Added BOM
Parts:
- F1, F2, F3, F4, F5, F6, F7, F8: Digi-Key PN (none) -> 36-3544-2-ND
- TB1: Digi-Key PN (none) -> ED2953-ND
Changed lines of the file:
@@
 F 2 "Barrier_Blocks:BARRIER_BLOCK_1ROW_2POS_P9.5MM" H 2750 2100 60  0001 C CNN
 F 3 "" H 2750 2100 60  0000 C CNN
+F 4 "ED2953-ND" H 2750 2100 50  0001 C CNN "Digi-Key PN"
 	1    2750 2100
 	-1   0    0    -1
@@
 F 7 "Fuse Clip; 500 VAC; 30 A; PCB; For 0.110 in. x 0.032 in. mini blade fuses" H 3650 2025 50  0001 L BNN "Field7"
 F 8 "Keystone Electronics" H 3650 2025 50  0001 L BNN "Field8"
+F 9 "36-3544-2-ND" H 4650 1800 50  0001 C CNN "Digi-Key PN"
 	1    4650 1800
 	1    0    0    -1
@@
 F 7 "Fuse Clip; 500 VAC; 30 A; PCB; For 0.110 in. x 0.032 in. mini blade fuses" H 3650 2125 50  0001 L BNN "Field7"
 F 8 "Keystone Electronics" H 3650 2125 50  0001 L BNN "Field8"
+F 9 "36-3544-2-ND" H 4650 1900 50  0001 C CNN "Digi-Key PN"
 	1    4650 1900
 	1    0    0    -1
@@
 F 7 "Fuse Clip; 500 VAC; 30 A; PCB; For 0.110 in. x 0.032 in. mini blade fuses" H 3650 2225 50  0001 L BNN "Field7"
 F 8 "Keystone Electronics" H 3650 2225 50  0001 L BNN "Field8"
+F 9 "36-3544-2-ND" H 4650 2000 50  0001 C CNN "Digi-Key PN"
 	1    4650 2000
 	1    0    0    -1
@@
 F 7 "Fuse Clip; 500 VAC; 30 A; PCB; For 0.110 in. x 0.032 in. mini blade fuses" H 3650 2325 50  0001 L BNN "Field7"
 F 8 "Keystone Electronics" H 3650 2325 50  0001 L BNN "Field8"
+F 9 "36-3544-2-ND" H 4650 2100 50  0001 C CNN "Digi-Key PN"
 	1    4650 2100
 	1    0    0    -1
@@
 F 7 "Fuse Clip; 500 VAC; 30 A; PCB; For 0.110 in. x 0.032 in. mini blade fuses" H 3650 2425 50  0001 L BNN "Field7"
 F 8 "Keystone Electronics" H 3650 2425 50  0001 L BNN "Field8"
+F 9 "36-3544-2-ND" H 4650 2200 50  0001 C CNN "Digi-Key PN"
 	1    4650 2200
 	1    0    0    -1
@@
 F 7 "Fuse Clip; 500 VAC; 30 A; PCB; For 0.110 in. x 0.032 in. mini blade fuses" H 3650 2525 50  0001 L BNN "Field7"
 F 8 "Keystone Electronics" H 3650 2525 50  0001 L BNN "Field8"
+F 9 "36-3544-2-ND" H 4650 2300 50  0001 C CNN "Digi-Key PN"
 	1    4650 2300
 	1    0    0    -1
@@
 F 7 "Fuse Clip; 500 VAC; 30 A; PCB; For 0.110 in. x 0.032 in. mini blade fuses" H 3650 2625 50  0001 L BNN "Field7"
 F 8 "Keystone Electronics" H 3650 2625 50  0001 L BNN "Field8"
+F 9 "36-3544-2-ND" H 4650 2400 50  0001 C CNN "Digi-Key PN"
 	1    4650 2400
 	1    0    0    -1
@@
 F 7 "Fuse Clip; 500 VAC; 30 A; PCB; For 0.110 in. x 0.032 in. mini blade fuses" H 3650 2725 50  0001 L BNN "Field7"
 F 8 "Keystone Electronics" H 3650 2725 50  0001 L BNN "Field8"
+F 9 "36-3544-2-ND" H 4650 2500 50  0001 C CNN "Digi-Key PN"
 	1    4650 2500
 	1    0    0    -1
