File: Pixel_Boost/Pixel_Boost.kicad_sch (KiCad schematic)
At the start: 9 parts, among them J1 In, J2 Out, U1 MCP1703A-SOT89, U2 74LVC1G17

Commit message: added logo
Other:
- title: (none) -> Pixel Boost
Changed lines of the file:
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@@
 (kicad_sch (version 20211123) (generator eeschema)
   (paper "A4")
+  (title_block
+    (title "Pixel Boost")
+    (date "2022-12-13")
+    (rev "v1")
+  )
   (junction (at 190.5 92.71) (diameter 0) (color 0 0 0 0)
   )
