File: Pixel_Boost/Pixel_Boost.kicad_sch (KiCad schematic)
At the start: 9 parts, among them J1 In, J2 Out, U1 MCP1703A-SOT89, U2 74LVC1G17

Commit message: change footprint
Parts:
- J1, J2: footprint Connector_Phoenix_MC:PhoenixContact_MCV_1,5_3-G-3.81_1x03_P3.81mm_Vertical -> Scotts:PhoenixContact_MCV_1,5_3-G-3.81_1x03_P3.81mm_Vertical
- U2: LCSC C840096 -> C7836
