File: PS2_Power_Breakout/PS2_Power_Breakout.kicad_sch (KiCad schematic)
At the start: 17 parts, among them J1 PJ-041H, J10 PJ-041H, J11 Neg Center, J12 PJ-041H, J2 Pos Center, J3 Pos Center, J4 Pos Center, J5 Pos Center, J6 Pos Center, J7 PJ-041H, J8 PJ-041H, J9 PJ-041H

Commit message: added digikey part numbers
Parts:
- J1, J10, J12, J7, J8, J9: Digi-Key_PN (none) -> CP-041H-ND; MPN (none) -> PJ-041H
Changed lines of the file:
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@@
       (effects (font (size 1.27 1.27)) (justify left bottom) hide)
+    )
+    (property "Digi-Key_PN" "CP-041H-ND" (at 167.64 88.9 0)
+      (effects (font (size 1.27 1.27)) hide)
+    )
+    (property "MPN" "PJ-041H" (at 167.64 88.9 0)
+      (effects (font (size 1.27 1.27)) hide)
     )
     (pin "1")
@@
       (effects (font (size 1.27 1.27)) (justify left bottom) hide)
     )
+    (property "Digi-Key_PN" "CP-041H-ND" (at 91.44 88.9 0)
+      (effects (font (size 1.27 1.27)) hide)
+    )
+    (property "MPN" "PJ-041H" (at 91.44 88.9 0)
+      (effects (font (size 1.27 1.27)) hide)
+    )
     (pin "1")
     (pin "2")
@@
     (property "MANUFACTURER" "CUI" (at 142.24 88.9 0)
       (effects (font (size 1.27 1.27)) (justify left bottom) hide)
+    )
+    (property "Digi-Key_PN" "CP-041H-ND" (at 142.24 88.9 0)
+      (effects (font (size 1.27 1.27)) hide)
+    )
+    (property "MPN" "PJ-041H" (at 142.24 88.9 0)
+      (effects (font (size 1.27 1.27)) hide)
     )
     (pin "1")
@@
       (effects (font (size 1.27 1.27)) (justify left bottom) hide)
     )
+    (property "Digi-Key_PN" "CP-041H-ND" (at 116.84 88.9 0)
+      (effects (font (size 1.27 1.27)) hide)
+    )
+    (property "MPN" "PJ-041H" (at 116.84 88.9 0)
+      (effects (font (size 1.27 1.27)) hide)
+    )
     (pin "1")
     (pin "2")
@@
       (effects (font (size 1.27 1.27)) (justify left bottom) hide)
     )
+    (property "Digi-Key_PN" "CP-041H-ND" (at 193.04 88.9 0)
+      (effects (font (size 1.27 1.27)) hide)
+    )
+    (property "MPN" "PJ-041H" (at 193.04 88.9 0)
+      (effects (font (size 1.27 1.27)) hide)
+    )
     (pin "1")
     (pin "2")
@@
       (effects (font (size 1.27 1.27)) (justify left bottom) hide)
     )
-    (pin "1")
+    (property "Digi-Key_PN" "CP-041H-ND" (at 38.1 76.2 0)
+      (effects (font (size 1.27 1.27)) hide)
+    )
+    (property "MPN" "PJ-041H" (at 38.1 76.2 0)
+      (effects (font (size 1.27 1.27)) hide)
+    )
+    (pin "1")
